File: Schematics/ArduCuff.sch (EAGLE design)
At the start: 22 parts, among them IC1 MEGA8-P, IC2 7805, IC3 KA78RH33, J1 POWER_JACKPTH_LOCK, J2 AVR_SPI_PRG_6NS, U1 HC_05, Y1 16MHZ

Commit message: sd
Parts:
- added U2: HEX_CONVERTER, SparkFun:HEX_CONVERTER
Connections:
- removed net N$12: IC1.PB5(SCK), J2.3
- removed net N$13: IC1.PB4(MISO), J2.1
- removed net N$14: IC1.PB3(MOSI/OC2), J2.4
- new net CSSD: U2.1A
- new net MISO: IC1.PB4(MISO), J2.1, U$2.DO
- new net MOSI: IC1.PB3(MOSI/OC2), J2.4, U2.2A
- new net N$10: U$2.DI, U2.2Y
- new net N$11: U2.3Y
- new net N$8: U$2.CS, U2.1Y
- new net SCK: IC1.PB5(SCK), J2.3, U2.3A
- net 3.3V: now also U$2.VCC, U2.VCC
- net GND: now also U$2.GND, U$2.GND1, U$2.SHIELD, U2.GND
- net RST: now also J2.5
